File: lasermodule/scanhead_pcb_compact/baseboard/fpga.kicad_sch (KiCad schematic)
At the start: 20 parts, among them U12 ICE40UP5K-SG48ITR-FPGA_Lattice, U13 S25FL064LABMFI010, U14 MCP1700x-120xxTT

Commit message: laid out board
Parts:
- U12: footprint Package_DFN_QFN:QFN-48-1EP_7x7mm_P0.5mm_EP5.6x5.6mm -> sockets_scanhead:QFN-48-1EP_7x7mm_P0.5mm_EP5.6x5.6mm
Connections:
- net CFG_DONE: no longer U12.46 (IOB_0a)
- net DIGITAL: now also U12.31 (IOT_42b); no longer U12.38 (IOT_50b)
- net HALL2: now also U12.32 (IOT_43a); no longer U12.36 (IOT_48b)
- net IC_HB_PWM1: now also U12.2 (IOB_6a); no longer U12.31 (IOT_42b)
- net IC_HB_PWM2: now also U12.3 (IOB_9b); no longer U12.28 (IOT_41a)
- net RGB0: now also D2.3 (GK); no longer D2.4 (BK)
- net RGB1: now also D2.2 (RK); no longer D2.3 (GK)
- net RGB2: now also D2.4 (BK); no longer D2.2 (RK)
- net SD_IO2: now also U12.21 (IOB_23b); no longer U12.10 (IOB_18a)
- net SPI_SCK: now also U12.19 (IOB_29b); no longer U12.18 (IOB_31b)
- net SPI_SI: now also U12.18 (IOB_31b); no longer U12.21 (IOB_23b)
- net SPI_SO: now also U12.13 (IOB_24a); no longer U12.19 (IOB_29b)
- net SPI_SS2: now also U12.12 (IOB_22a); no longer U12.13 (IOB_24a)
- net X_PO: now also U12.11 (IOB_20a); no longer U12.3 (IOB_9b)
- net uH: now also U12.43 (IOT_49a); no longer U12.26 (IOT_39a)
- net uL: now also U12.44 (IOB_3b_G6); no longer U12.25 (IOT_36b)
- net vH: now also U12.45 (IOB_5b); no longer U12.23 (IOT_37a)
- net vL: now also U12.46 (IOB_0a); no longer U12.9 (IOB_16a)
- net wH: now also U12.47 (IOB_2a); no longer U12.32 (IOT_43a)
- net wL: now also U12.48 (IOB_4a); no longer U12.27 (IOT_38b)
- no-connect marks 10 -> 11
