File: lasermodule/scanhead_pcb_compact/baseboard/laserhead.kicad_sch (KiCad schematic)
At the start: 42 parts, among them J3 Conn_01x02, J4 Conn_01x03, J5 Conn_01x02, J6 jumper wire 2 pin, U1 DIGIPOT_50K, U11 LM7808_TO220, U2 U_IC-HKB, U3 STSPIN230, U4 MIC920, U5 MIC920, U6 DRV5033FAxDBZ, U7 DRV5033FAxDBZ, U8 DRV5033FAxDBZ

Commit message: laid out board
Parts:
- removed R16, R17, R18: Zero, Resistor_SMD:R_0805_2012Metric_Pad1.20x1.40mm_HandSolder, symbol Device:R
Connections:
- net u: now also U3.3 (OUTU)
- net v: now also U3.8 (OUTV)
- net w: now also U3.10 (OUTW)
Other:
- moved on the sheet: J4
Changed lines of the file:
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@@
     (stroke (width 0) (type default))
   )
-  (text "pcb motor" (at 93.98 100.33 0)
+  (text "pcb motor" (at 96.52 72.39 0)
     (effects (font (size 1.27 1.27)) (justify left bottom))
   )
@@
     )
   )
-  (global_label "u" (shape input) (at 100.33 90.17 0) (fields_autoplaced)
+  (global_label "u" (shape input) (at 102.87 62.23 0) (fields_autoplaced)
     (effects (font (size 1.27 1.27)) (justify left))
-    (property "Intersheetrefs" "${INTERSHEET_REFS}" (at 103.7306 90.17 0)
+    (property "Intersheetrefs" "${INTERSHEET_REFS}" (at 106.2706 62.23 0)
       (effects (font (size 1.27 1.27)) (justify left) hide)
     )
@@
     )
   )
-  (global_label "u" (shape input) (at 87.63 50.8 0) (fields_autoplaced)
+  (global_label "u" (shape input) (at 80.01 50.8 0) (fields_autoplaced)
     (effects (font (size 1.27 1.27)) (justify left))
-    (property "Intersheetrefs" "${INTERSHEET_REFS}" (at 91.0306 50.8 0)
+    (property "Intersheetrefs" "${INTERSHEET_REFS}" (at 83.4106 50.8 0)
       (effects (font (size 1.27 1.27)) (justify left) hide)
     )
@@
     )
   )
-  (global_label "v" (shape input) (at 100.33 92.71 0) (fields_autoplaced)
+  (global_label "v" (shape input) (at 102.87 64.77 0) (fields_autoplaced)
     (effects (font (size 1.27 1.27)) (justify left))
-    (property "Intersheetrefs" "${INTERSHEET_REFS}" (at 103.5492 92.71 0)
+    (property "Intersheetrefs" "${INTERSHEET_REFS}" (at 106.0892 64.77 0)
       (effects (font (size 1.27 1.27)) (justify left) hide)
     )
   )
-  (global_label "w" (shape input) (at 100.33 95.25 0) (fields_autoplaced)
+  (global_label "w" (shape input) (at 102.87 67.31 0) (fields_autoplaced)
     (effects (font (size 1.27 1.27)) (justify left))
-    (property "Intersheetrefs" "${INTERSHEET_REFS}" (at 103.9121 95.25 0)
+    (property "Intersheetrefs" "${INTERSHEET_REFS}" (at 106.4521 67.31 0)
       (effects (font (size 1.27 1.27)) (justify left) hide)
     )
@@
     )
   )
-  (global_label "v" (shape input) (at 87.63 58.42 0) (fields_autoplaced)
+  (global_label "v" (shape input) (at 80.01 58.42 0) (fields_autoplaced)
     (effects (font (size 1.27 1.27)) (justify left))
-    (property "Intersheetrefs" "${INTERSHEET_REFS}" (at 90.8492 58.42 0)
+    (property "Intersheetrefs" "${INTERSHEET_REFS}" (at 83.2292 58.42 0)
       (effects (font (size 1.27 1.27)) (justify left) hide)
     )
   )
-  (global_label "w" (shape input) (at 87.63 66.04 0) (fields_autoplaced)
+  (global_label "w" (shape input) (at 80.01 66.04 0) (fields_autoplaced)
     (effects (font (size 1.27 1.27)) (justify left))
-    (property "Intersheetrefs" "${INTERSHEET_REFS}" (at 91.2121 66.04 0)
+    (property "Intersheetrefs" "${INTERSHEET_REFS}" (at 83.5921 66.04 0)
       (effects (font (size 1.27 1.27)) (justify left) hide)
-    )
-  )
-  (symbol (lib_id "Device:R") (at 83.82 50.8 90) (unit 1)
-    (in_bom yes) (on_board yes) (dnp no)
-    (property "Reference" "R16" (at 83.82 53.34 90)
-      (effects (font (size 1.27 1.27)))
-    )
-    (property "Value" "Zero" (at 82.55 48.26 90)
-      (effects (font (size 1.27 1.27)))
-    )
-    (property "Footprint" "Resistor_SMD:R_0805_2012Metric_Pad1.20x1.40mm_HandSolder" (at 83.82 52.578 90)
-      (effects (font (size 1.27 1.27)) hide)
-    )
-    (property "Datasheet" "~" (at 83.82 50.8 0)
-      (effects (font (size 1.27 1.27)) hide)
-    )
-    (pin "1")
-    (pin "2")
-    (instances
-      (project "scanhead_pcb"
-        (path "/e63e39d7-6ac0-4ffd-8aa3-1841a4541b55/a3ece103-0834-4f34-b268-bf200f179698"
-          (reference "R16") (unit 1)
-        )
-      )
     )
   )
@@
     )
   )
-  (symbol (lib_id "Device:R") (at 83.82 66.04 90) (unit 1)
-    (in_bom yes) (on_board yes) (dnp no)
-    (property "Reference" "R18" (at 83.82 68.58 90)
-      (effects (font (size 1.27 1.27)))
-    )
-    (property "Value" "Zero" (at 82.55 63.5 90)
-      (effects (font (size 1.27 1.27)))
-    )
-    (property "Footprint" "Resistor_SMD:R_0805_2012Metric_Pad1.20x1.40mm_HandSolder" (at 83.82 67.818 90)
-      (effects (font (size 1.27 1.27)) hide)
-    )
-    (property "Datasheet" "~" (at 83.82 66.04 0)
-      (effects (font (size 1.27 1.27)) hide)
-    )
-    (pin "1")
-    (pin "2")
-    (instances
-      (project "scanhead_pcb"
-        (path "/e63e39d7-6ac0-4ffd-8aa3-1841a4541b55/a3ece103-0834-4f34-b268-bf200f179698"
-          (reference "R18") (unit 1)
-        )
-      )
-    )
-  )
   (symbol (lib_id "Device:R") (at 137.16 52.07 180) (unit 1)
     (in_bom yes) (on_board yes) (dnp no)
@@
     )
   )
-  (symbol (lib_id "Device:R") (at 83.82 58.42 90) (unit 1)
-    (in_bom yes) (on_board yes) (dnp no)
-    (property "Reference" "R17" (at 83.82 60.96 90)
-      (effects (font (size 1.27 1.27)))
-    )
-    (property "Value" "Zero" (at 82.55 55.88 90)
-      (effects (font (size 1.27 1.27)))
-    )
-    (property "Footprint" "Resistor_SMD:R_0805_2012Metric_Pad1.20x1.40mm_HandSolder" (at 83.82 60.198 90)
-      (effects (font (size 1.27 1.27)) hide)
-    )
-    (property "Datasheet" "~" (at 83.82 58.42 0)
-      (effects (font (size 1.27 1.27)) hide)
-    )
-    (pin "1")
-    (pin "2")
-    (instances
-      (project "scanhead_pcb"
-        (path "/e63e39d7-6ac0-4ffd-8aa3-1841a4541b55/a3ece103-0834-4f34-b268-bf200f179698"
-          (reference "R17") (unit 1)
-        )
-      )
-    )
-  )
   (symbol (lib_id "power:GND") (at 210.82 127 90) (unit 1)
     (in_bom yes) (on_board yes) (dnp no)
@@
     )
   )
-  (symbol (lib_id "Connector_Generic:Conn_01x03") (at 95.25 92.71 180) (unit 1)
+  (symbol (lib_id "Connector_Generic:Conn_01x03") (at 97.79 64.77 180) (unit 1)
     (in_bom yes) (on_board yes) (dnp no) (fields_autoplaced)
-    (property "Reference" "J4" (at 95.25 83.82 0)
-      (effects (font (size 1.27 1.27)))
-    )
-    (property "Value" "Conn_01x03" (at 95.25 86.36 0)
-      (effects (font (size 1.27 1.27)))
-    )
-    (property "Footprint" "Connector_PinHeader_2.54mm:PinHeader_1x03_P2.54mm_Vertical" (at 95.25 92.71 0)
-      (effects (font (size 1.27 1.27)) hide)
-    )
-    (property "Datasheet" "~" (at 95.25 92.71 0)
-      (effects (font (size 1.27 1.27)) hide)
-    )
+    (property "Reference" "J4" (at 97.79 55.88 0)
+      (effects (font (size 1.27 1.27)))
+    )
+    (property "Value" "Conn_01x03" (at 97.79 58.42 0)
+      (effects (font (size 1.27 1.27)))
+    )
+    (property "Footprint" "Connector_PinHeader_2.54mm:PinHeader_1x03_P2.54mm_Vertical" (at 97.79 64.77 0)
+      (effects (font (size 1.27 1.27)) hide)
+    )
+    (property "Datasheet" "~" (at 97.79 64.77 0)
+      (effects (font (size 1.27 1.27)) hide)
+    )
