File: lasermodule/base/base.kicad_pcb (KiCad board)
At the start: 2 copper layers, 107.2 x 60 mm, 64 parts, among them J1 Connector_Generic_Conn_01x02, J2 FPC 15 pin molex vertical, J3 Conn_01x02, J4 Conn_01x03, J5 Conn_01x02, J6 jumper wire 2 pin, U1 DIGIPOT_50K, U10 MCP1700x-330xxTT, U11 LM7808_TO220, U12 ICE40UP5K-SG48ITR-FPGA_Lattice, U13 S25FL064LABMFI010, U14 MCP1700x-120xxTT, U2 U_IC-HKB, U3 STSPIN230, U4 MIC920, U5 MIC920, U6 DRV5033FAxDBZ, U7 DRV5033FAxDBZ, U8 DRV5033FAxDBZ, U9 LM7805_TO220

Commit message: added pcbmotor, renamed some folders
Parts:
- J4: footprint Connector_PinHeader_2.54mm:PinHeader_1x03_P2.54mm_Vertical -> sockets_scanhead:pcbmotor_smd
Changed lines of the file:
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@@
   (net 60 "unconnected-(U12A-IOT_48b-Pad36)")
   (net 61 "unconnected-(U12A-IOT_37a-Pad23)")
-  (net 62 "Net-(D1-K)")
+  (net 62 "Net-(#FLG0103-pwr)")
   (footprint "Package_TO_SOT_THT:TO-220-3_Vertical" (layer "F.Cu")
     (at 153.2352 126.1042 180)
@@
       (net 61 "unconnected-(U12A-IOT_37a-Pad23)") (pinfunction "IOT_37a") (pintype "bidirectional+no_connect"))
     (pad "24" smd roundrect (at 2.75 3.9375 180) (size 0.25 1.875) (layers "F.Cu" "F.Paste" "F.Mask") (roundrect_rratio 0.25)
-      (net 62 "Net-(D1-K)") (pinfunction "VPP_2V5") (pintype "power_in"))
+      (net 62 "Net-(#FLG0103-pwr)") (pinfunction "VPP_2V5") (pintype "power_in"))
     (pad "25" smd roundrect (at 3.9375 2.75 180) (size 1.875 0.25) (layers "F.Cu" "F.Paste" "F.Mask") (roundrect_rratio 0.25)
       (net 55 "unconnected-(U12A-IOT_36b-Pad25)") (pinfunction "IOT_36b") (pintype "bidirectional+no_connect"))
@@
     )
   )
-  (footprint "Connector_PinHeader_2.54mm:PinHeader_1x03_P2.54mm_Vertical" (layer "F.Cu")
+  (footprint "sockets_scanhead:pcbmotor_smd" (layer "F.Cu")
     (at 80.896 112.637)
     (descr "Through hole straight pin header, 1x03, 2.54mm pitch, single row")
@@
         (effects (font (size 1 1) (thickness 0.15)))
     )
-    (fp_text value "Conn_01x03" (at 0 7.41) (layer "F.Fab")
+    (fp_text value "Conn_01x03" (at 0 10.8458) (layer "F.Fab")
         (effects (font (size 1 1) (thickness 0.15)))
     )
@@
     (fp_line (start -1.33 1.27) (end -1.33 6.41)
       (stroke (width 0.12) (type solid)) (layer "F.SilkS"))
-    (fp_line (start -1.33 1.27) (end 1.33 1.27)
-      (stroke (width 0.12) (type solid)) (layer "F.SilkS"))
     (fp_line (start -1.33 6.41) (end 1.33 6.41)
       (stroke (width 0.12) (type solid)) (layer "F.SilkS"))
-    (fp_line (start 1.33 1.27) (end 1.33 6.41)
+    (fp_line (start 1.339802 -1.27) (end 1.33 6.41)
       (stroke (width 0.12) (type solid)) (layer "F.SilkS"))
     (fp_line (start -1.8 -1.8) (end -1.8 6.85)
@@
     (fp_line (start 1.27 6.35) (end -1.27 6.35)
       (stroke (width 0.1) (type solid)) (layer "F.Fab"))
-    (pad "1" thru_hole rect (at 0 0) (size 1.7 1.7) (drill 1) (layers "*.Cu" "*.Mask")
+    (pad "1" smd rect (at 0 0) (size 1.7 1.7) (layers "F.Cu" "F.Paste" "F.Mask")
       (net 37 "w") (pinfunction "Pin_1") (pintype "passive"))
-    (pad "2" thru_hole oval (at 0 2.54) (size 1.7 1.7) (drill 1) (layers "*.Cu" "*.Mask")
+    (pad "2" smd rect (at 0 2.54) (size 1.7 1.7) (layers "F.Cu" "F.Paste" "F.Mask")
       (net 38 "v") (pinfunction "Pin_2") (pintype "passive"))
-    (pad "3" thru_hole oval (at 0 5.08) (size 1.7 1.7) (drill 1) (layers "*.Cu" "*.Mask")
+    (pad "3" smd rect (at 0 5.08) (size 1.7 1.7) (layers "F.Cu" "F.Paste" "F.Mask")
       (net 39 "u") (pinfunction "Pin_3") (pintype "passive"))
-    (model "${KICAD6_3DMODEL_DIR}/Connector_PinHeader_2.54mm.3dshapes/PinHeader_1x03_P2.54mm_Vertical.wrl"
-      (offset (xyz 0 0 0))
-      (scale (xyz 1 1 1))
-      (rotate (xyz 0 0 0))
-    )
   )
   (footprint "Capacitor_SMD:C_0805_2012Metric_Pad1.18x1.45mm_HandSolder" (layer "F.Cu")
@@
       (stroke (width 0.1) (type solid)) (layer "F.Fab"))
     (pad "1" smd roundrect (at -2.5 0 90) (size 3.5 1.8) (layers "F.Cu" "F.Paste" "F.Mask") (roundrect_rratio 0.1388888889)
-      (net 62 "Net-(D1-K)") (pinfunction "K") (pintype "passive"))
+      (net 62 "Net-(#FLG0103-pwr)") (pinfunction "K") (pintype "passive"))
     (pad "2" smd roundrect (at 2.5 0 90) (size 3.5 1.8) (layers "F.Cu" "F.Paste" "F.Mask") (roundrect_rratio 0.1388888889)
       (net 12 "+3V3") (pinfunction "A") (pintype "passive"))
@@
         (xy 126.192411 115.994243)
         (xy 126.252093 115.070978)
-        (xy 126.272 114.146)
       )
     )

Commit message: further cleaned up and tested renders in blender
Parts:
- D2: footprint LED_SMD:LED_Cree-PLCC4_2x2mm_CW -> sockets_scanhead:LED_Cree-PLCC4_2x2mm_CW
- J1: footprint Connector_AMASS:AMASS_XT30PW-F_1x02_P2.50mm_Horizontal -> sockets_scanhead:AMASS_XT30PW-F_1x02_P2.50mm_Horizontal
- U13: footprint Package_SO:SOIC-8W_5.3x5.3mm_P1.27mm -> sockets_scanhead:SOIC-8W_5.3x5.3mm_P1.27mm
- U3: footprint Package_DFN_QFN:VQFN-16-1EP_3x3mm_P0.5mm_EP1.8x1.8mm -> sockets_scanhead:VQFN-16-1EP_3x3mm_P0.5mm_EP1.8x1.8mm
- moved J4 1.51 mm to (80.9, 114.1)
Routing:
- net w: track 68.6 -> 69.7 mm
- net v: track 67.8 -> 68.8 mm
- net u: track 58.4 -> 59.5 mm
Other:
- board text added: "PCB3D_BR_base"
- board text added: "PCB3D_TL_base"
