File: lasermodule/pcbmotor/pcbmotor.kicad_sch (KiCad schematic)
At the start: 1 part, among them J1 Conn_01x03

Commit message: further cleaned up and tested renders in blender
Parts:
- J1: footprint Connector_PinHeader_2.54mm:PinHeader_1x03_P2.54mm_Vertical -> pcbmotor:PinHeader_1x03_P2.54mm_Vertical
Changed lines of the file:
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@@
       (effects (font (size 1.27 1.27)))
     )
-    (property "Footprint" "Connector_PinHeader_2.54mm:PinHeader_1x03_P2.54mm_Vertical" (at 50.8 36.83 0)
+    (property "Footprint" "pcbmotor:PinHeader_1x03_P2.54mm_Vertical" (at 50.8 36.83 0)
       (effects (font (size 1.27 1.27)) hide)
     )
@@
     (pin "3")
     (instances
-      (project "scanhead_pcb"
+      (project "pcbmotor"
         (path "/e63e39d7-6ac0-4ffd-8aa3-1841a4541b55"
           (reference "J1") (unit 1)
