File: lasermodule/frontplate/frontplate.kicad_sch (KiCad schematic)
At the start: 2 parts

Commit message: simplified loading in freecad, updated pcbs
Parts:
- L1, L2: value (none) -> Logo_Open_Hardware_Large; footprint (none) -> footprints:hexastorm
Changed lines of the file:
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@@
-(kicad_sch (version 20211123) (generator eeschema)
+(kicad_sch (version 20230121) (generator eeschema)
   (paper "A4")
   (text "hexastorm front" (at 138.43 90.17 0)
@@
   )
   (symbol (lib_id "Graphic:Logo_Open_Hardware_Large") (at 144.78 105.41 0) (unit 1)
-    (in_bom yes) (on_board yes)
-    (property "Reference" "L1" (id 0) (at 144.78 92.71 0)
+    (in_bom yes) (on_board yes) (dnp no)
+    (property "Reference" "L1" (at 144.78 92.71 0)
       (effects (font (size 1.27 1.27)) hide)
     )
-    (property "Value" "" (id 1) (at 144.78 115.57 0)
+    (property "Value" "Logo_Open_Hardware_Large" (at 144.78 115.57 0)
       (effects (font (size 1.27 1.27)) hide)
     )
-    (property "Footprint" "" (id 2) (at 144.78 105.41 0)
+    (property "Footprint" "footprints:hexastorm" (at 144.78 105.41 0)
       (effects (font (size 1.27 1.27)) hide)
     )
-    (property "Datasheet" "~" (id 3) (at 144.78 105.41 0)
+    (property "Datasheet" "~" (at 144.78 105.41 0)
       (effects (font (size 1.27 1.27)) hide)
+    )
+    (instances
+      (project "frontplate"
+        (path "/85697c89-1348-441e-add9-eb5a39865876"
+          (reference "L1") (unit 1)
+        )
+      )
     )
   )
   (symbol (lib_id "Graphic:Logo_Open_Hardware_Large") (at 143.51 73.66 0) (unit 1)
-    (in_bom yes) (on_board yes)
-    (property "Reference" "L2" (id 0) (at 143.51 60.96 0)
+    (in_bom yes) (on_board yes) (dnp no)
+    (property "Reference" "L2" (at 143.51 60.96 0)
       (effects (font (size 1.27 1.27)) hide)
     )
-    (property "Value" "" (id 1) (at 143.51 83.82 0)
+    (property "Value" "Logo_Open_Hardware_Large" (at 143.51 83.82 0)
       (effects (font (size 1.27 1.27)) hide)
     )
-    (property "Footprint" "" (id 2) (at 143.51 73.66 0)
+    (property "Footprint" "footprints:hexastorm" (at 143.51 73.66 0)
       (effects (font (size 1.27 1.27)) hide)
     )
-    (property "Datasheet" "~" (id 3) (at 143.51 73.66 0)
+    (property "Datasheet" "~" (at 143.51 73.66 0)
       (effects (font (size 1.27 1.27)) hide)
+    )
+    (instances
+      (project "frontplate"
+        (path "/85697c89-1348-441e-add9-eb5a39865876"
+          (reference "L2") (unit 1)
+        )
+      )
     )
   )
@@
     (path "/" (page "1"))
   )
-  (symbol_instances
-    (path "/00000000-0000-0000-0000-00006168343a"
-      (reference "L1") (unit 1) (value "Logo_Open_Hardware_Large") (footprint "footprints:hexastorm")
-    )
-    (path "/00000000-0000-0000-0000-000061683d03"
-      (reference "L2") (unit 1) (value "Logo_Open_Hardware_Large") (footprint "footprints:hexastorm")
-    )
-  )
 )
